File: windsensor/schematics/windsensor-esp12-v002.sch (EAGLE design)
At the start: 15 parts, among them IC1 MCP1700TT3302, IC3 HAL556, T1 JC501

Commit message: changed output capacitor from 1µ to 10µ to increase voltage stability
Parts:
- C2: value 1µ -> 10µ
Changed lines of the file:
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@@
 <part name="GND12" library="supply1" deviceset="GND" device=""/>
 <part name="C1" library="rcl" deviceset="C-EU" device="C0805" value="1µ"/>
-<part name="C2" library="rcl" deviceset="C-EU" device="C0805" value="1µ"/>
+<part name="C2" library="rcl" deviceset="C-EU" device="C0805" value="10µ"/>
 <part name="GND8" library="supply1" deviceset="GND" device=""/>
 <part name="GND14" library="supply1" deviceset="GND" device=""/>
